Commit message: fixed URFD WITH SOLIDWORKSgit add .

File: src/robot_description/urdf/Assembly-Robot-URDF.urdf.xacro (robot description, xacro)
@@ -4,5 +4,5 @@
      For more information, please see http://wiki.ros.org/sw_urdf_exporter -->
 <robot
-  name="autonomous_robot_description">
+  name="robot_description">
   <link name="base_footprint">
       <origin xyz="0 0 0" rpy="0 0 0" />
@@ -34,18 +34,14 @@
         rpy="0 0 0" />
       <geometry>
-          <mesh filename="package://autonomous_robot_description/meshes/base_link.stl"/>
-      </geometry>
-      <material
-        name="">
-        <color
-          rgba="0.752941176470588 0.752941176470588 0.752941176470588 1" />
-      </material>
-    </visual>
-    <collision>
-      <origin
-        xyz="0 0 0"
-        rpy="0 0 0" />
-      <geometry>
-        <mesh filename="package://autonomous_robot_description/meshes/base_link.stl"/>
+          <mesh filename="file:///home/tamir/autonomousPro/src/robot_description/meshes/base_link.stl" scale="1 1 1"/>
+      </geometry>
+      <material name="grey"/>
+    </visual>
+    <collision>
+      <origin
+        xyz="0 0 0"
+        rpy="0 0 0" />
+      <geometry>
+        <mesh filename="file:///home/tamir/autonomousPro/src/robot_description/meshes/base_link.stl" scale="1 1 1"/>
       </geometry>
     </collision>
@@ -72,18 +68,14 @@
         rpy="0 0 0" />
       <geometry>
-      <mesh filename="package://autonomous_robot_description/meshes/front_hinge.stl" />
-      </geometry>
-      <material
-        name="">
-        <color
-          rgba="0.792156862745098 0.819607843137255 0.933333333333333 1" />
-      </material>
-    </visual>
-    <collision>
-      <origin
-        xyz="0 0 0"
-        rpy="0 0 0" />
-      <geometry>
-      <mesh filename="package://autonomous_robot_description/meshes/front_hinge.stl" />
+      <mesh filename="file:///home/tamir/autonomousPro/src/robot_description/meshes/front_hinge.stl" scale="1 1 1"/>
+      </geometry>
+      <material name="grey"/>
+    </visual>
+    <collision>
+      <origin
+        xyz="0 0 0"
+        rpy="0 0 0" />
+      <geometry>
+      <mesh filename="file:///home/tamir/autonomousPro/src/robot_description/meshes/front_hinge.stl" scale="1 1 1"/>
       </geometry>
     </collision>
@@ -130,18 +122,14 @@
         rpy="0 0 0" />
       <geometry>
-          <mesh filename="package://autonomous_robot_description/meshes/front_wheel_link.stl" />
-      </geometry>
-      <material
-        name="">
-        <color
-          rgba="0.792156862745098 0.819607843137255 0.933333333333333 1" />
-      </material>
-    </visual>
-    <collision>
-      <origin
-        xyz="0 0 0"
-        rpy="0 0 0" />
-      <geometry>
-         <mesh filename="package://autonomous_robot_description/meshes/front_wheel_link.stl" />
+          <mesh filename="file:///home/tamir/autonomousPro/src/robot_description/meshes/front_wheel_link.stl" scale="1 1 1"/>
+      </geometry>
+      <material name="black"/>
+    </visual>
+    <collision>
+      <origin
+        xyz="0 0 0"
+        rpy="0 0 0" />
+      <geometry>
+         <mesh filename="file:///home/tamir/autonomousPro/src/robot_description/meshes/front_wheel_link.stl" scale="1 1 1"/>
       </geometry>
     </collision>
@@ -181,18 +169,14 @@
         rpy="0 0 0" />
       <geometry>
-      <mesh filename="package://autonomous_robot_description/meshes/left_wheel_link.stl" />
-      </geometry>
-      <material
-        name="">
-        <color
-          rgba="0.752941176470588 0.752941176470588 0.752941176470588 1" />
-      </material>
-    </visual>
-    <collision>
-      <origin
-        xyz="0 0 0"
-        rpy="0 0 0" />
-      <geometry>
-          <mesh filename="package://autonomous_robot_description/meshes/left_wheel_link.stl" />
+      <mesh filename="file:///home/tamir/autonomousPro/src/robot_description/meshes/left_wheel_link.stl" scale="1 1 1"/>
+      </geometry>
+      <material name="black"/>
+    </visual>
+    <collision>
+      <origin
+        xyz="0 0 0"
+        rpy="0 0 0" />
+      <geometry>
+          <mesh filename="file:///home/tamir/autonomousPro/src/robot_description/meshes/left_wheel_link.stl" scale="1 1 1"/>
       </geometry>
     </collision>
@@ -237,18 +221,14 @@
         rpy="0 0 0" />
       <geometry>
-          <mesh filename="package://autonomous_robot_description/meshes/rear_hinge.stl" />
-      </geometry>
-      <material
-        name="">
-        <color
-          rgba="0.792156862745098 0.819607843137255 0.933333333333333 1" />
-      </material>
-    </visual>
-    <collision>
-      <origin
-        xyz="0 0 0"
-        rpy="0 0 0" />
-      <geometry>
-          <mesh filename="package://autonomous_robot_description/meshes/rear_hinge.stl" />
+          <mesh filename="file:///home/tamir/autonomousPro/src/robot_description/meshes/rear_hinge.stl" scale="1 1 1"/>
+      </geometry>
+      <material name="grey"/>
+    </visual>
+    <collision>
+      <origin
+        xyz="0 0 0"
+        rpy="0 0 0" />
+      <geometry>
+          <mesh filename="file:///home/tamir/autonomousPro/src/robot_description/meshes/rear_hinge.stl" scale="1 1 1"/>
       </geometry>
     </collision>
@@ -295,18 +275,14 @@
         rpy="0 0 0" />
       <geometry>
-        <mesh filename="package://autonomous_robot_description/meshes/rear_wheel_link.stl" />
-      </geometry>
-      <material
-        name="">
-        <color
-          rgba="0.792156862745098 0.819607843137255 0.933333333333333 1" />
-      </material>
-    </visual>
-    <collision>
-      <origin
-        xyz="0 0 0"
-        rpy="0 0 0" />
-      <geometry>
-         <mesh filename="package://autonomous_robot_description/meshes/rear_wheel_link.stl" />
+        <mesh filename="file:///home/tamir/autonomousPro/src/robot_description/meshes/rear_wheel_link.stl" scale="1 1 1"/>
+      </geometry>
+      <material name="black"/>
+    </visual>
+    <collision>
+      <origin
+        xyz="0 0 0"
+        rpy="0 0 0" />
+      <geometry>
+         <mesh filename="file:///home/tamir/autonomousPro/src/robot_description/meshes/rear_wheel_link.stl" scale="1 1 1"/>
       </geometry>
     </collision>
@@ -346,18 +322,14 @@
         rpy="0 0 0" />
       <geometry>
-          <mesh filename="package://autonomous_robot_description/meshes/right_wheel_link.stl" />
-      </geometry>
-      <material
-        name="">
-        <color
-          rgba="0.752941176470588 0.752941176470588 0.752941176470588 1" />
-      </material>
-    </visual>
-    <collision>
-      <origin
-        xyz="0 0 0"
-        rpy="0 0 0" />
-      <geometry>
-          <mesh filename="package://autonomous_robot_description/meshes/right_wheel_link.stl" />
+          <mesh filename="file:///home/tamir/autonomousPro/src/robot_description/meshes/right_wheel_link.stl" scale="1 1 1"/>
+      </geometry>
+      <material name="black"/>
+    </visual>
+    <collision>
+      <origin
+        xyz="0 0 0"
+        rpy="0 0 0" />
+      <geometry>
+          <mesh filename="file:///home/tamir/autonomousPro/src/robot_description/meshes/right_wheel_link.stl" scale="1 1 1"/>
       </geometry>
     </collision>
@@ -402,18 +374,14 @@
         rpy="0 0 0" />
       <geometry>
-          <mesh filename="package://autonomous_robot_description/meshes/camera_link.stl" />
-      </geometry>
-      <material
-        name="">
-        <color
-          rgba="1 1 1 1" />
-      </material>
-    </visual>
-    <collision>
-      <origin
-        xyz="0 0 0"
-        rpy="0 0 0" />
-      <geometry>
-        <mesh filename="package://autonomous_robot_description/meshes/camera_link.stl" />
+          <mesh filename="file:///home/tamir/autonomousPro/src/robot_description/meshes/camera_link.stl" scale="1 1 1"/>
+      </geometry>
+      <material name="yellow"/>
+    </visual>
+    <collision>
+      <origin
+        xyz="0 0 0"
+        rpy="0 0 0" />
+      <geometry>
+        <mesh filename="file:///home/tamir/autonomousPro/src/robot_description/meshes/camera_link.stl" scale="1 1 1"/>
       </geometry>
     </collision>
@@ -453,18 +421,14 @@
         rpy="0 0 0" />
       <geometry>
-          <mesh filename="package://autonomous_robot_description/meshes/lidar_link.stl" />
-      </geometry>
-      <material
-        name="">
-        <color
-          rgba="0.00784313725490196 0.23921568627451 0.823529411764706 1" />
-      </material>
-    </visual>
-    <collision>
-      <origin
-        xyz="0 0 0"
-        rpy="0 0 0" />
-      <geometry>
-          <mesh filename="package://autonomous_robot_description/meshes/lidar_link.stl" />
+          <mesh filename="file:///home/tamir/autonomousPro/src/robot_description/meshes/lidar_link.stl" scale="1 1 1"/>
+      </geometry>
+      <material name="cyan"/>
+    </visual>
+    <collision>
+      <origin
+        xyz="0 0 0"
+        rpy="0 0 0" />
+      <geometry>
+          <mesh filename="file:///home/tamir/autonomousPro/src/robot_description/meshes/lidar_link.stl" scale="1 1 1"/>
       </geometry>
     </collision>
@@ -483,3 +447,79 @@
       xyz="0 0 0" />
   </joint>
+    <link name="imu_link"/>
+  <joint name="base_to_imu" type="fixed">
+    <parent link="base_link"/>
+    <child  link="imu_link"/>
+    <origin xyz="0 0 0" rpy="0 0 0"/>
+  </joint>
+      <!-- Gazebo Plugin for IMU -->
+    <gazebo reference="imu_link">
+        <sensor name="imu_sensor" type="imu">
+            <always_on>true</always_on>
+            <visualize>true</visualize>
+            <update_rate>100.0</update_rate>
+            <plugin name="imu_controller" filename="libgazebo_ros_imu_sensor.so">
+                <ros>
+                    <argument>~/out:=imu</argument> <!--   the topic we are publishing on    -->
+                </ros>
+                <output_type>sensor_msgs/msg/Imu</output_type>
+                <frame_name>imu_link</frame_name>
+            </plugin>
+            <imu>
+                <topic>/imu</topic>
+                <gaussian_noise>0.01</gaussian_noise>
+            </imu>
+        </sensor>
+    </gazebo>
+        <!-- Gazebo Plugin for Lidar -->
+    <gazebo reference="lidar_link">
+        <sensor name="laser_link" type="ray">
+            <pose> 0 0 0 0 0 0 </pose>
+            <visualize>true</visualize>
+            <update_rate>20.0</update_rate>
+            <ray>
+                <scan>
+                    <horizontal>
+                        <samples>500</samples>
+                        <min_angle>-3.14</min_angle>
+                        <max_angle>3.14</max_angle>
+                    </horizontal>
+                </scan>
+                <range>
+                    <min>0.5</min>
+                    <max>10</max>
+                </range>
+            </ray>
+            <plugin name="laser_controller" filename="libgazebo_ros_ray_sensor.so">
+                <ros>
+                    <argument>~/out:=scan</argument>   <!-- the topic we are publishing on -->
+                </ros>
+                <output_type>sensor_msgs/msg/LaserScan</output_type>
+                <frame_name>lidar_link</frame_name>
+            </plugin>
+        </sensor>
+    </gazebo>
+        <!-- Gazebo Plugin for Camera -->
+    <gazebo reference="camera_link">
+        <sensor name="camera_sensor" type="camera">
+            <pose>0 0 0 0 0 0</pose>
+            <visualize>true</visualize>
+            <update_rate>10.0</update_rate>
+            <camera>
+                <horizontal_fov>1.047</horizontal_fov>
+                <image>
+                    <format>B8G8R8</format>
+                    <width>640</width>
+                    <height>480</height>
+                </image>
+                <clip>
+                    <near>0.05</near>
+                    <far>8.0</far>
+                </clip>
+            </camera>
+            <plugin name="camera_controller" filename="libgazebo_ros_camera.so">
+                <frame_name>camera_link_optical</frame_name>
+            </plugin>
+        </sensor>
+    </gazebo>
 </robot>

File: src/robot_description/urdf/autonomous_robot.urdf.xacro (robot description, xacro)
@@ -4,6 +4,6 @@
     <xacro:arg name="sim_mode" default="true"/>
     <xacro:include filename="common_properties.xacro" />
-    <xacro:include filename="mobile_robot.xacro" />
-    <!-- <xacro:include filename="Assembly-Robot-URDF.urdf.xacro" /> -->
+    <xacro:include filename="Assembly-Robot-URDF.urdf.xacro" />
+    <!-- <xacro:include filename="mobile_robot.xacro" /> -->
 <!-- switching between ros2_control and gazebo control -->
     <xacro:if value="$(arg use_ros2_control)">
@@ -13,7 +13,7 @@
         <xacro:include filename="autonomous_robot_gazebo.xacro" />
     </xacro:unless>
-    <xacro:include filename="imu.xacro" />
+    <!-- <xacro:include filename="imu.xacro" />
     <xacro:include filename="lidar.xacro" />
     <xacro:include filename="camera.xacro" />
-    <xacro:include filename="gazebo_color.xacro" />
+    <xacro:include filename="gazebo_color.xacro" /> -->
 </robot>

File: src/robot_description/urdf/autonomous_robot_gazebo.xacro (robot description, xacro)
@@ -8,5 +8,6 @@
             <left_joint>left_wheel_joint</left_joint>
             <right_joint>right_wheel_joint</right_joint>
-            <wheel_separation>0.48</wheel_separation>
+            <!-- kinematics -->
+            <wheel_separation>0.7</wheel_separation>
             <wheel_diameter>0.16</wheel_diameter>
             <!-- limits -->

File: src/robot_description/urdf/common_properties.xacro (robot description, xacro)
@@ -1,45 +1,47 @@
 <?xml version="1.0"?>
 <robot xmlns:xacro="http://www.ros.org/wiki/xacro">
-    <material name="grey">
-        <color rgba="0.5 0.5 0.5 1" />
-    </material>
-    <material name="green">
-        <color rgba="0 0.5 0 1" />
-    </material>
-    <material name="blue">
-        <color rgba="0 0 1 1" />
-    </material>
-    <material name="pink">
-        <color rgba="1 0 1 1" />
-    </material>
-    <material name="yellow">
-        <color rgba="0.5 0.5 0 1" />
-    </material>
-    <material name="orange">
-        <color rgba="1 0.5 0 1" />
-    </material>
-    <material name="red">
-        <color rgba="1 0 0.2 1" />
-    </material>
-    <material name="black">
-        <color rgba="0 0 0 1" />
-    </material>
-    <xacro:macro name="box_inertia" params="mass l w h xyz rpy">
-        <inertial>
-            <origin xyz="${xyz}" rpy="0 0 0" />
-            <mass value="${mass}" />
-            <inertia ixx="${mass/12 * (h*h + l*l)}" ixy="0" ixz="0"
-                     iyy="${mass/12 * (w*w + l*l)}" iyz="0"
-                     izz="${mass/12 * (h*h + w*w)}" />
-        </inertial>
-    </xacro:macro>
-    <xacro:macro name="wheel_inertia" params="mass l r xyz rpy">
-        <inertial>
-            <origin xyz="${xyz}" rpy="${rpy}" />
-            <mass value="${mass}" />
-            <inertia ixx="${mass/12 * (3*r*r + l*l)}" ixy="0" ixz="0"
-                     iyy="${mass/12 * (3*r*r + l*l)}" iyz="0"
-                     izz="${mass/2 * (r*r)}" />
-        </inertial>
-    </xacro:macro>
+  <!-- Matches RViz gray on base_link -->
+  <material name="grey">
+    <color rgba="0.752941 0.752941 0.752941 1"/>
+  </material>
+  <!-- Light blue used for front_hinge & rear_hinge -->
+  <material name="blue">
+    <color rgba="0.792157 0.819608 0.933333 1"/>
+  </material>
+  <!-- Wheels dark gray/black -->
+  <material name="black">
+    <color rgba="0.1 0.1 0.1 1"/>
+  </material>
+  <!-- Camera pale yellow -->
+  <material name="yellow">
+    <color rgba="1 0.95 0.6 1"/>
+  </material>
+  <!-- Lidar light blue -->
+  <material name="cyan">
+    <color rgba="0.6 0.8 1 1"/>
+  </material>
+  <!-- Keep other colors available (not used by current URDF visuals) -->
+  <material name="green"><color rgba="0 0.5 0 1"/></material>
+  <material name="pink"><color rgba="1 0 1 1"/></material>
+  <material name="orange"><color rgba="1 0.5 0 1"/></material>
+  <material name="red"><color rgba="1 0 0.2 1"/></material>
+  <!-- inertia macros unchanged -->
+  <xacro:macro name="box_inertia" params="mass l w h xyz rpy">
+    <inertial>
+      <origin xyz="${xyz}" rpy="0 0 0" />
+      <mass value="${mass}" />
+      <inertia ixx="${mass/12 * (h*h + l*l)}" ixy="0" ixz="0"
+               iyy="${mass/12 * (w*w + l*l)}" iyz="0"
+               izz="${mass/12 * (h*h + w*w)}" />
+    </inertial>
+  </xacro:macro>
+  <xacro:macro name="wheel_inertia" params="mass l r xyz rpy">
+    <inertial>
+      <origin xyz="${xyz}" rpy="${rpy}" />
+      <mass value="${mass}" />
+      <inertia ixx="${mass/12 * (3*r*r + l*l)}" ixy="0" ixz="0"
+               iyy="${mass/12 * (3*r*r + l*l)}" iyz="0"
+               izz="${mass/2 * (r*r)}" />
+    </inertial>
+  </xacro:macro>
 </robot>

File: src/robot_description/urdf/lidar.xacro (robot description, xacro)
@@ -21,5 +21,5 @@
         <parent link="base_link" />
         <child link="lidar_link" />
-        <origin xyz="${base_l / 4.0} 0 ${(base_h / 2.0) + (lidar_h / 2.0)}" rpy="0 0 -1.507" />
+        <origin xyz="${base_l / 4.0} 0 ${(base_h / 2.0) + (lidar_h / 2.0)}" rpy="0 0 0" />
     </joint>
     <gazebo reference ="lidar_link">

File: src/robot_description/urdf/ros2_control.xacro (robot description, xacro)
@@ -56,5 +56,5 @@
     <gazebo>
         <plugin name="gazebo_ros2_control" filename="libgazebo_ros2_control.so">
-           <parameters>package://autonomous_robot_description/config/joint_controller.yaml</parameters>
+            <parameters>$(find robot_description)/config/joint_controller.yaml</parameters>
         </plugin>
     </gazebo>

Commit message: updated hinges and depth camera

File: src/robot_description/urdf/Assembly-Robot-URDF.urdf.xacro (robot description, xacro)
@@ -6,10 +6,10 @@
   name="robot_description">
   <link name="base_footprint">
-      <origin xyz="0 0 0" rpy="0 0 0" />
+      <origin xyz="0 0 0.1" rpy="0 0 0" />
   </link>
   <joint name="base_footprint_to_base_link" type="fixed">
     <parent link="base_footprint"/>
     <child link="base_link"/>
-    <origin xyz="0 0 0.45" rpy="0 0 0"/>
+    <origin xyz="0 0 0.4" rpy="0 0 0"/>
   </joint>
   <link
@@ -85,5 +85,5 @@
     type="revolute">
     <origin
-      xyz="0.48615 3E-05 -0.249"
+      xyz="0.48615 3E-05 -0.2385"
       rpy="0 0 0" />
     <parent
@@ -99,5 +99,5 @@
       velocity="10" />
     <dynamics
-      friction="0.1" />
+      friction="0.0" />
   </joint>
   <link
@@ -238,5 +238,5 @@
     type="revolute">
     <origin
-      xyz="-0.47385 3E-05 -0.249"
+      xyz="-0.47385 3E-05 -0.2385"
       rpy="0 0 0" />
     <parent
@@ -252,5 +252,5 @@
       velocity="10" />
     <dynamics
-      friction="0.1" />
+      friction="0.0" />
   </joint>
   <link
@@ -500,12 +500,11 @@
         </sensor>
     </gazebo>
-        <!-- Gazebo Plugin for Camera -->
     <gazebo reference="camera_link">
-        <sensor name="camera_sensor" type="camera">
-            <pose>0 0 0 0 0 0</pose>
+        <sensor name="camera" type="depth">
+            <pose> 0 0 0 0 0 0 </pose>
             <visualize>true</visualize>
-            <update_rate>10.0</update_rate>
+            <update_rate>10</update_rate>
             <camera>
-                <horizontal_fov>1.047</horizontal_fov>
+                <horizontal_fov>1.089</horizontal_fov>
                 <image>
                     <format>B8G8R8</format>
@@ -520,4 +519,6 @@
             <plugin name="camera_controller" filename="libgazebo_ros_camera.so">
                 <frame_name>camera_link_optical</frame_name>
+                <min_depth>0.1</min_depth>
+                <max_depth>100.0</max_depth>
             </plugin>
         </sensor>
