Commit message: changed the path for the mtl

File: src/robot_description/urdf/Assembly-Robot-URDF.urdf.xacro (robot description, xacro)
@@ -34,5 +34,5 @@
         rpy="0 0 0" />
       <geometry>
-          <mesh filename="file:///home/tamir/autonomousPro/src/robot_description/meshes/base_link.stl" scale="1 1 1"/>
+          <mesh filename="file:///home/tamir/thesis/autonomousPro/src/robot_description/meshes/base_link.stl" scale="1 1 1"/>
       </geometry>
       <material name="grey"/>
@@ -43,5 +43,5 @@
         rpy="0 0 0" />
       <geometry>
-        <mesh filename="file:///home/tamir/autonomousPro/src/robot_description/meshes/base_link.stl" scale="1 1 1"/>
+        <mesh filename="file:///home/tamir/thesis/autonomousPro/src/robot_description/meshes/base_link.stl" scale="1 1 1"/>
       </geometry>
     </collision>
@@ -68,5 +68,5 @@
         rpy="0 0 0" />
       <geometry>
-      <mesh filename="file:///home/tamir/autonomousPro/src/robot_description/meshes/front_hinge.stl" scale="1 1 1"/>
+      <mesh filename="file:///home/tamir/thesis/autonomousPro/src/robot_description/meshes/front_hinge.stl" scale="1 1 1"/>
       </geometry>
       <material name="grey"/>
@@ -77,5 +77,5 @@
         rpy="0 0 0" />
       <geometry>
-      <mesh filename="file:///home/tamir/autonomousPro/src/robot_description/meshes/front_hinge.stl" scale="1 1 1"/>
+      <mesh filename="file:///home/tamir/thesis/autonomousPro/src/robot_description/meshes/front_hinge.stl" scale="1 1 1"/>
       </geometry>
     </collision>
@@ -122,5 +122,5 @@
         rpy="0 0 0" />
       <geometry>
-          <mesh filename="file:///home/tamir/autonomousPro/src/robot_description/meshes/front_wheel_link.stl" scale="1 1 1"/>
+          <mesh filename="file:///home/tamir/thesis/autonomousPro/src/robot_description/meshes/front_wheel_link.stl" scale="1 1 1"/>
       </geometry>
       <material name="black"/>
@@ -131,5 +131,5 @@
         rpy="0 0 0" />
       <geometry>
-         <mesh filename="file:///home/tamir/autonomousPro/src/robot_description/meshes/front_wheel_link.stl" scale="1 1 1"/>
+         <mesh filename="file:///home/tamir/thesis/autonomousPro/src/robot_description/meshes/front_wheel_link.stl" scale="1 1 1"/>
       </geometry>
     </collision>
@@ -169,5 +169,5 @@
         rpy="0 0 0" />
       <geometry>
-      <mesh filename="file:///home/tamir/autonomousPro/src/robot_description/meshes/left_wheel_link.stl" scale="1 1 1"/>
+      <mesh filename="file:///home/tamir/thesis/autonomousPro/src/robot_description/meshes/left_wheel_link.stl" scale="1 1 1"/>
       </geometry>
       <material name="black"/>
@@ -178,5 +178,5 @@
         rpy="0 0 0" />
       <geometry>
-          <mesh filename="file:///home/tamir/autonomousPro/src/robot_description/meshes/left_wheel_link.stl" scale="1 1 1"/>
+          <mesh filename="file:///home/tamir/thesis/autonomousPro/src/robot_description/meshes/left_wheel_link.stl" scale="1 1 1"/>
       </geometry>
     </collision>
@@ -221,5 +221,5 @@
         rpy="0 0 0" />
       <geometry>
-          <mesh filename="file:///home/tamir/autonomousPro/src/robot_description/meshes/rear_hinge.stl" scale="1 1 1"/>
+          <mesh filename="file:///home/tamir/thesis/autonomousPro/src/robot_description/meshes/rear_hinge.stl" scale="1 1 1"/>
       </geometry>
       <material name="grey"/>
@@ -230,5 +230,5 @@
         rpy="0 0 0" />
       <geometry>
-          <mesh filename="file:///home/tamir/autonomousPro/src/robot_description/meshes/rear_hinge.stl" scale="1 1 1"/>
+          <mesh filename="file:///home/tamir/thesis/autonomousPro/src/robot_description/meshes/rear_hinge.stl" scale="1 1 1"/>
       </geometry>
     </collision>
@@ -275,5 +275,5 @@
         rpy="0 0 0" />
       <geometry>
-        <mesh filename="file:///home/tamir/autonomousPro/src/robot_description/meshes/rear_wheel_link.stl" scale="1 1 1"/>
+        <mesh filename="file:///home/tamir/thesis/autonomousPro/src/robot_description/meshes/rear_wheel_link.stl" scale="1 1 1"/>
       </geometry>
       <material name="black"/>
@@ -284,5 +284,5 @@
         rpy="0 0 0" />
       <geometry>
-         <mesh filename="file:///home/tamir/autonomousPro/src/robot_description/meshes/rear_wheel_link.stl" scale="1 1 1"/>
+         <mesh filename="file:///home/tamir/thesis/autonomousPro/src/robot_description/meshes/rear_wheel_link.stl" scale="1 1 1"/>
       </geometry>
     </collision>
@@ -322,5 +322,5 @@
         rpy="0 0 0" />
       <geometry>
-          <mesh filename="file:///home/tamir/autonomousPro/src/robot_description/meshes/right_wheel_link.stl" scale="1 1 1"/>
+          <mesh filename="file:///home/tamir/thesis/autonomousPro/src/robot_description/meshes/right_wheel_link.stl" scale="1 1 1"/>
       </geometry>
       <material name="black"/>
@@ -331,5 +331,5 @@
         rpy="0 0 0" />
       <geometry>
-          <mesh filename="file:///home/tamir/autonomousPro/src/robot_description/meshes/right_wheel_link.stl" scale="1 1 1"/>
+          <mesh filename="file:///home/tamir/thesis/autonomousPro/src/robot_description/meshes/right_wheel_link.stl" scale="1 1 1"/>
       </geometry>
     </collision>
@@ -374,5 +374,5 @@
         rpy="0 0 0" />
       <geometry>
-          <mesh filename="file:///home/tamir/autonomousPro/src/robot_description/meshes/camera_link.stl" scale="1 1 1"/>
+          <mesh filename="file:///home/tamir/thesis/autonomousPro/src/robot_description/meshes/camera_link.stl" scale="1 1 1"/>
       </geometry>
       <material name="yellow"/>
@@ -383,5 +383,5 @@
         rpy="0 0 0" />
       <geometry>
-        <mesh filename="file:///home/tamir/autonomousPro/src/robot_description/meshes/camera_link.stl" scale="1 1 1"/>
+        <mesh filename="file:///home/tamir/thesis/autonomousPro/src/robot_description/meshes/camera_link.stl" scale="1 1 1"/>
       </geometry>
     </collision>
@@ -421,5 +421,5 @@
         rpy="0 0 0" />
       <geometry>
-          <mesh filename="file:///home/tamir/autonomousPro/src/robot_description/meshes/lidar_link.stl" scale="1 1 1"/>
+          <mesh filename="file:///home/tamir/thesis/autonomousPro/src/robot_description/meshes/lidar_link.stl" scale="1 1 1"/>
       </geometry>
       <material name="cyan"/>
@@ -430,5 +430,5 @@
         rpy="0 0 0" />
       <geometry>
-          <mesh filename="file:///home/tamir/autonomousPro/src/robot_description/meshes/lidar_link.stl" scale="1 1 1"/>
+          <mesh filename="file:///home/tamir/thesis/autonomousPro/src/robot_description/meshes/lidar_link.stl" scale="1 1 1"/>
       </geometry>
     </collision>
